Commit message: refactored lidar urdf description

File: description/urdf/diffbot.urdf.xacro (robot description, xacro)
@@ -8,5 +8,4 @@
   <!-- Import diffbot ros2_control description -->
   <xacro:include filename="$(find hoverboard_driver)/ros2_control/hoverboard_driver.ros2_control.xacro" />
-  <!-- Import lidar description -->
   <xacro:diffbot prefix="$(arg prefix)" />
   <xacro:hoverboard_driver_ros2_control

File: description/urdf/diffbot_description.urdf.xacro (robot description, xacro)
@@ -166,28 +166,6 @@
   <link name="base_footprint">
   </link>
-<joint name="lidar_joint" type="fixed">
-  <parent link="${prefix}base_link"/>
-  <child link="lidar_link"/>
-  <origin xyz="-0.30 0 0.20" rpy="0 0 0"/>
-</joint>
-  <link name="lidar_link">
-    <inertial>
-      <origin xyz="0 0 0" rpy="0 0 0"/>
-      <mass value="0.125"/>
-      <inertia ixx="0.001"  ixy="0"  ixz="0" iyy="0.001" iyz="0" izz="0.001" />
-    </inertial>
-    <collision>
-      <origin xyz="0 0 0" rpy="0 0 0"/>
-      <geometry>
-        <cylinder radius="0.0508" length="0.055"/>
-      </geometry>
-    </collision>
-    <visual>
-      <origin xyz="0 0 0" rpy="0 0 0"/>
-      <geometry>
-        <cylinder radius="0.0508" length="0.055"/>
-      </geometry>
-    </visual>
-  </link>
+  <!-- Include Lidar -->
+  <xacro:include filename="$(find hoverboard_driver)/urdf/lidar.xacro" />
   </xacro:macro>
 </robot>

File: description/urdf/lidar.xacro (robot description, xacro)
@@ -2,27 +2,27 @@
 <robot xmlns:xacro="http://www.ros.org/wiki/xacro" >
 <joint name="lidar_joint" type="fixed">
-  <parent link="base_link"/>
+  <parent link="${prefix}base_link"/>
   <child link="lidar_link"/>
-  <origin xyz="0 0 0.12" rpy="0 0 0"/>
+  <origin xyz="0.30 0 0.20" rpy="0 0 ${PI}"/>
 </joint>
-<link name="lidar_link">
-  <inertial>
-    <origin xyz="0 0 0" rpy="0 0 0"/>
-    <mass value="0.125"/>
-    <inertia ixx="0.001"  ixy="0"  ixz="0" iyy="0.001" iyz="0" izz="0.001" />
-  </inertial>
-  <collision>
-    <origin xyz="0 0 0" rpy="0 0 0"/>
-    <geometry>
-       <cylinder radius="0.0508" length="0.055"/>
-    </geometry>
-  </collision>
-  <visual>
-    <origin xyz="0 0 0" rpy="0 0 0"/>
-    <geometry>
-       <cylinder radius="0.0508" length="0.055"/>
-    </geometry>
-  </visual>
-</link>
+  <link name="lidar_link">
+    <inertial>
+      <origin xyz="0 0 0" rpy="0 0 0"/>
+      <mass value="0.125"/>
+      <inertia ixx="0.001"  ixy="0"  ixz="0" iyy="0.001" iyz="0" izz="0.001" />
+    </inertial>
+    <collision>
+      <origin xyz="0 0 0" rpy="0 0 0"/>
+      <geometry>
+        <cylinder radius="0.0508" length="0.055"/>
+      </geometry>
+    </collision>
+    <visual>
+      <origin xyz="0 0 0" rpy="0 0 0"/>
+      <geometry>
+        <cylinder radius="0.0508" length="0.055"/>
+      </geometry>
+    </visual>
+  </link>
 <gazebo reference="lidar_link">
   <sensor name="lidar" type="ray">
