Commit message: fixed lidar yaw and angles for gazebo sim

File: description/urdf/lidar.xacro (robot description, xacro)
@@ -4,5 +4,5 @@
   <parent link="${prefix}base_link"/>
   <child link="lidar_link"/>
-  <origin xyz="0.30 0 0.20" rpy="0 0 ${PI}"/>
+  <origin xyz="0.30 0 0.20" rpy="0 0 0"/>
 </joint>
   <link name="lidar_link">
@@ -35,6 +35,6 @@
           <samples>360</samples>
           <resolution>1.000000</resolution>
-          <min_angle>0.000000</min_angle>
-          <max_angle>6.280000</max_angle>
+          <min_angle>-1.0472</min_angle>
+          <max_angle>1.0472</max_angle>
         </horizontal>
       </scan>
