Commit message: added gazebo materials

File: description/urdf/diffbot_description.urdf.xacro (robot description, xacro)
@@ -38,4 +38,7 @@
       </inertial>
     </link>
+    <gazebo reference="${prefix}base_link">
+      <material>Gazebo/Orange</material>
+    </gazebo>
     <joint name="${prefix}left_wheel_joint" type="continuous">
       <parent link="${prefix}base_link"/>
@@ -69,4 +72,7 @@
         </inertial>
       </link>
+      <gazebo reference="${prefix}left_wheel">
+          <material>Gazebo/Black</material>
+      </gazebo>
     <joint name="${prefix}right_wheel_joint" type="continuous">
       <parent link="${prefix}base_link"/>
@@ -100,4 +106,7 @@
         </inertial>
       </link>
+      <gazebo reference="${prefix}right_wheel">
+          <material>Gazebo/Black</material>
+      </gazebo>
     <joint name="${prefix}caster_frontal_wheel_joint" type="fixed">
       <parent link="${prefix}base_link"/>
@@ -134,4 +143,9 @@
       <origin xyz="${-base_width/2 + caster_wheel_radius} 0 -0.045" rpy="0 0 0"/>
     </joint>
+    <gazebo reference="${prefix}caster_frontal_wheel">
+        <material>Gazebo/White</material>
+        <mu1 value="0.001"/>
+        <mu2 value="0.001"/>
+    </gazebo>
     <!-- caster rear wheel Link -->
     <link name="${prefix}caster_rear_wheel">
@@ -158,4 +172,9 @@
         </inertial>
       </link>
+      <gazebo reference="${prefix}caster_rear_wheel">
+        <material>Gazebo/White</material>
+        <mu1 value="0.001"/>
+        <mu2 value="0.001"/>
+      </gazebo>
   <!-- BASE_FOOTPRINT LINK -->
   <joint name="base_footprint_joint" type="fixed">

Commit message: wheels changes

File: description/urdf/diffbot_description.urdf.xacro (robot description, xacro)
@@ -109,72 +109,6 @@
           <material>Gazebo/Black</material>
       </gazebo>
-    <joint name="${prefix}caster_frontal_wheel_joint" type="fixed">
-      <parent link="${prefix}base_link"/>
-      <child link="${prefix}caster_frontal_wheel"/>
-      <origin xyz="${base_width/2 - caster_wheel_radius} 0 -0.045" rpy="0 0 0"/>
-    </joint>
-    <!-- caster frontal wheel Link -->
-    <link name="${prefix}caster_frontal_wheel">
-      <collision>
-        <origin xyz="0 0 0" rpy="0 0 0"/>
-        <geometry>
-          <sphere radius="${caster_wheel_radius}"/>
-        </geometry>
-      </collision>
-      <visual>
-        <origin xyz="0 0 0" rpy="0 0 0"/>
-        <geometry>
-          <sphere radius="${caster_wheel_radius}"/>
-        </geometry>
-        <material name="white"/>
-      </visual>
-      <inertial>
-        <origin xyz="0 0 0" rpy="0 0 0"/>
-        <mass value="${caster_wheel_mass}"/>
-        <inertia
-          ixx="${caster_wheel_mass * 0.4 * (caster_wheel_radius * caster_wheel_radius)}" ixy="0.0" ixz="0.0"
-          iyy="${caster_wheel_mass * 0.4 * (caster_wheel_radius * caster_wheel_radius)}" iyz="0.0"
-          izz="${caster_wheel_mass * 0.4 * (caster_wheel_radius * caster_wheel_radius)}"/>
-        </inertial>
-      </link>
-    <joint name="${prefix}caster_rear_wheel_joint" type="fixed">
-      <parent link="${prefix}base_link"/>
-      <child link="${prefix}caster_rear_wheel"/>
-      <origin xyz="${-base_width/2 + caster_wheel_radius} 0 -0.045" rpy="0 0 0"/>
-    </joint>
-    <gazebo reference="${prefix}caster_frontal_wheel">
-        <material>Gazebo/White</material>
-        <mu1 value="0.001"/>
-        <mu2 value="0.001"/>
-    </gazebo>
-    <!-- caster rear wheel Link -->
-    <link name="${prefix}caster_rear_wheel">
-      <collision>
-        <origin xyz="0 0 0" rpy="0 0 0"/>
-        <geometry>
-          <sphere radius="${caster_wheel_radius}"/>
-        </geometry>
-      </collision>
-      <visual>
-        <origin xyz="0 0 0" rpy="0 0 0"/>
-        <geometry>
-          <sphere radius="${caster_wheel_radius}"/>
-        </geometry>
-        <material name="white"/>
-      </visual>
-      <inertial>
-        <origin xyz="0 0 0" rpy="0 0 0"/>
-        <mass value="${caster_wheel_mass}"/>
-        <inertia
-          ixx="${caster_wheel_mass * 0.4 * (caster_wheel_radius * caster_wheel_radius)}" ixy="0.0" ixz="0.0"
-          iyy="${caster_wheel_mass * 0.4 * (caster_wheel_radius * caster_wheel_radius)}" iyz="0.0"
-          izz="${caster_wheel_mass * 0.4 * (caster_wheel_radius * caster_wheel_radius)}"/>
-        </inertial>
-      </link>
-      <gazebo reference="${prefix}caster_rear_wheel">
-        <material>Gazebo/White</material>
-        <mu1 value="0.001"/>
-        <mu2 value="0.001"/>
-      </gazebo>
+  <!-- Include Caster Wheels -->
+  <xacro:include filename="$(find hoverboard_driver)/urdf/caster_wheels.urdf.xacro"/>
   <!-- BASE_FOOTPRINT LINK -->
   <joint name="base_footprint_joint" type="fixed">
