Commit message: lots

File: description/urdf/caster_wheels.urdf.xacro (robot description, xacro)
@@ -14,5 +14,5 @@
           <sphere radius="${caster_wheel_radius}"/>
         </geometry>
-        <material name="white"/>
+        <material name="green"/>
       </visual>
       <inertial>
@@ -25,5 +25,5 @@
       </inertial>
       <gazebo reference="${prefix}caster_frontal_left_wheel">
-        <material>Gazebo/White</material>
+        <material>Gazebo/Green</material>
         <mu1 value="0.001"/>
         <mu2 value="0.001"/>
@@ -43,5 +43,5 @@
           <sphere radius="${caster_wheel_radius}"/>
         </geometry>
-        <material name="white"/>
+        <material name="green"/>
       </visual>
       <inertial>
@@ -54,5 +54,5 @@
       </inertial>
       <gazebo reference="${prefix}caster_frontal_right_wheel">
-        <material>Gazebo/White</material>
+        <material>Gazebo/Green</material>
         <mu1 value="0.001"/>
         <mu2 value="0.001"/>
@@ -63,5 +63,5 @@
       <parent link="${prefix}base_link"/>
       <child link="${prefix}caster_frontal_left_wheel"/>
-      <origin xyz="${-base_width/2 + caster_wheel_radius} ${base_width/2} -0.045" rpy="0 0 0"/>
+      <origin xyz="${base_width/2} ${base_width/2 - caster_wheel_radius} -0.045" rpy="0 0 0"/>
     </joint>
     <!-- Caster Frontal Right Wheel Joint -->
@@ -69,5 +69,75 @@
       <parent link="${prefix}base_link"/>
       <child link="${prefix}caster_frontal_right_wheel"/>
-      <origin xyz="${-base_width/2 + caster_wheel_radius} ${-base_width/2} -0.045" rpy="0 0 0"/>
+      <origin xyz="${base_width/2} ${-base_width/2 + caster_wheel_radius} -0.045" rpy="0 0 0"/>
+    </joint>
+    <!-- Caster Rear Left Wheel Link -->
+    <link name="${prefix}caster_rear_left_wheel">
+      <collision>
+        <origin xyz="0 0 0" rpy="0 0 0"/>
+        <geometry>
+          <sphere radius="${caster_wheel_radius}"/>
+        </geometry>
+      </collision>
+      <visual>
+        <origin xyz="0 0 0" rpy="0 0 0"/>
+        <geometry>
+          <sphere radius="${caster_wheel_radius}"/>
+        </geometry>
+        <material name="green"/>
+      </visual>
+      <inertial>
+        <origin xyz="0 0 0" rpy="0 0 0"/>
+        <mass value="${caster_wheel_mass}"/>
+        <inertia
+          ixx="${caster_wheel_mass * 0.4 * (caster_wheel_radius * caster_wheel_radius)}" ixy="0.0" ixz="0.0"
+          iyy="${caster_wheel_mass * 0.4 * (caster_wheel_radius * caster_wheel_radius)}" iyz="0.0"
+          izz="${caster_wheel_mass * 0.4 * (caster_wheel_radius * caster_wheel_radius)}"/>
+      </inertial>
+      <gazebo reference="${prefix}caster_rear_left_wheel">
+        <material>Gazebo/Green</material>
+        <mu1 value="0.001"/>
+        <mu2 value="0.001"/>
+      </gazebo>
+    </link>
+    <!-- Caster Frontal Right Wheel Link -->
+    <link name="${prefix}caster_rear_right_wheel">
+      <collision>
+        <origin xyz="0 0 0" rpy="0 0 0"/>
+        <geometry>
+          <sphere radius="${caster_wheel_radius}"/>
+        </geometry>
+      </collision>
+      <visual>
+        <origin xyz="0 0 0" rpy="0 0 0"/>
+        <geometry>
+          <sphere radius="${caster_wheel_radius}"/>
+        </geometry>
+        <material name="green"/>
+      </visual>
+      <inertial>
+        <origin xyz="0 0 0" rpy="0 0 0"/>
+        <mass value="${caster_wheel_mass}"/>
+        <inertia
+          ixx="${caster_wheel_mass * 0.4 * (caster_wheel_radius * caster_wheel_radius)}" ixy="0.0" ixz="0.0"
+          iyy="${caster_wheel_mass * 0.4 * (caster_wheel_radius * caster_wheel_radius)}" iyz="0.0"
+          izz="${caster_wheel_mass * 0.4 * (caster_wheel_radius * caster_wheel_radius)}"/>
+      </inertial>
+      <gazebo reference="${prefix}caster_rear_right_wheel">
+        <material>Gazebo/Green</material>
+        <mu1 value="0.001"/>
+        <mu2 value="0.001"/>
+      </gazebo>
+    </link>
+    <!-- Caster Frontal Left Wheel Joint -->
+    <joint name="${prefix}caster_rear_left_wheel_joint" type="fixed">
+      <parent link="${prefix}base_link"/>
+      <child link="${prefix}caster_rear_left_wheel"/>
+      <origin xyz="${-base_width/2} ${base_width/2 - caster_wheel_radius} -0.045" rpy="0 0 0"/>
+    </joint>
+    <!-- Caster Frontal Right Wheel Joint -->
+    <joint name="${prefix}caster_rear_right_wheel_joint" type="fixed">
+      <parent link="${prefix}base_link"/>
+      <child link="${prefix}caster_rear_right_wheel"/>
+      <origin xyz="${-base_width/2} ${-base_width/2 + caster_wheel_radius} -0.045" rpy="0 0 0"/>
     </joint>
 </robot>

File: description/urdf/diffbot_description.urdf.xacro (robot description, xacro)
@@ -17,5 +17,5 @@
   <link name="${prefix}base_link">
     <collision>
-      <origin xyz="0 0 0" rpy="0 0 0"/>
+      <origin xyz="0 0 ${base_height/2}" rpy="0 0 0"/>
       <geometry>
         <box size="${base_width} ${base_length} ${base_height}"/>

File: description/urdf/lidar.xacro (robot description, xacro)
@@ -4,5 +4,5 @@
   <parent link="${prefix}base_link"/>
   <child link="lidar_link"/>
-  <origin xyz="0.30 0 0.20" rpy="0 0 ${PI}"/>
+  <origin xyz="${base_width/2} 0 -0.023" rpy="0 0 ${PI}"/>
 </joint>
   <link name="lidar_link">
@@ -15,5 +15,5 @@
       <origin xyz="0 0 0" rpy="0 0 0"/>
       <geometry>
-        <cylinder radius="0.0508" length="0.055"/>
+        <cylinder radius="0.0508" length="0.047"/>
       </geometry>
     </collision>
@@ -21,5 +21,5 @@
       <origin xyz="0 0 0" rpy="0 0 0"/>
       <geometry>
-        <cylinder radius="0.0508" length="0.055"/>
+        <cylinder radius="0.0508" length="0.047"/>
       </geometry>
     </visual>
@@ -35,6 +35,10 @@
           <samples>360</samples>
           <resolution>1.000000</resolution>
+          <min_angle>0</min_angle>
+          <max_angle>6.280000</max_angle>
+        <!--
           <min_angle>-1.0472</min_angle>
           <max_angle>1.0472</max_angle>
+        -->
         </horizontal>
       </scan>
