Commit message: minor fixes

File: description/ros2_control/hoverboard_driver.ros2_control.xacro (robot description, xacro)
@@ -6,5 +6,5 @@
         <plugin>hoverboard_driver/hoverboard_driver</plugin>
         <param name="wheel_radius">0.0825</param>
-        <param name="max_velocity">1.0</param>
+        <param name="max_velocity">0.5</param>
         <param name="device">/dev/serial/by-id/usb-1a86_USB_Serial-if00-port0</param>
       </hardware>

File: description/urdf/diffbot_description.urdf.xacro (robot description, xacro)
@@ -10,5 +10,5 @@
   <xacro:property name="wheel_mass" value="0.3" /> <!-- arbitrary value for wheel mass -->
   <xacro:property name="wheel_len" value="0.053" />
-  <xacro:property name="wheel_radius" value="0.085" />
+  <xacro:property name="wheel_radius" value="0.0825" />
   <xacro:property name="caster_wheel_mass" value="0.1" /> <!-- arbitrary value for caster wheel mass -->
   <xacro:property name="caster_wheel_radius" value="0.04" />

Commit message: general fixes and changes in params

File: description/ros2_control/hoverboard_driver.ros2_control.xacro (robot description, xacro)
@@ -2,22 +2,53 @@
 <robot xmlns:xacro="http://www.ros.org/wiki/xacro">
   <xacro:macro name="hoverboard_driver_ros2_control" params="name prefix">
-    <ros2_control name="${name}" type="system">
-      <hardware>
-        <plugin>hoverboard_driver/hoverboard_driver</plugin>
-        <param name="wheel_radius">0.0825</param>
-        <param name="max_velocity">0.5</param>
-        <param name="device">/dev/serial/by-id/usb-1a86_USB_Serial-if00-port0</param>
-      </hardware>
-      <joint name="${prefix}left_wheel_joint">
-        <command_interface name="velocity"/>
-        <state_interface name="position"/>
-        <state_interface name="velocity"/>
-      </joint>
-      <joint name="${prefix}right_wheel_joint">
-        <command_interface name="velocity"/>
-        <state_interface name="position"/>
-        <state_interface name="velocity"/>
-      </joint>
-    </ros2_control>
+    <xacro:unless value="$(arg sim_mode)">
+      <ros2_control name="${name}" type="system">
+        <hardware>
+          <plugin>hoverboard_driver/hoverboard_driver</plugin>
+          <param name="wheel_radius">0.0825</param>
+          <param name="max_velocity">2.5</param>  <!-- m/s -->
+          <param name="device">/dev/serial/by-id/usb-Prolific_Technology_Inc._USB-Serial_Controller-if00-port0</param>
+        </hardware>
+        <joint name="${prefix}left_wheel_joint">
+          <command_interface name="velocity"/>
+          <state_interface name="position"/>
+          <state_interface name="velocity"/>
+        </joint>
+        <joint name="${prefix}right_wheel_joint">
+          <command_interface name="velocity"/>
+          <state_interface name="position"/>
+          <state_interface name="velocity"/>
+        </joint>
+      </ros2_control>
+    </xacro:unless>
+    <xacro:if value="$(arg sim_mode)">
+      <ros2_control name="GazeboSystem" type="system">
+          <hardware>
+              <plugin>gazebo_ros2_control/GazeboSystem</plugin>
+          </hardware>
+          <joint name="left_wheel_joint">
+              <command_interface name="velocity">
+                  <param name="min">-10</param>
+                  <param name="max">10</param>
+              </command_interface>
+              <state_interface name="velocity"/>
+              <state_interface name="position"/>
+          </joint>
+          <joint name="right_wheel_joint">
+              <command_interface name="velocity">
+                  <param name="min">-10</param>
+                  <param name="max">10</param>
+              </command_interface>
+              <state_interface name="velocity"/>
+              <state_interface name="position"/>
+          </joint>
+      </ros2_control>
+    </xacro:if>
+    <gazebo>
+        <plugin name="gazebo_ros2_control" filename="libgazebo_ros2_control.so">
+            <parameters>$(find hoverboard_driver)/config/hoverboard_controllers.yaml</parameters>
+            <parameters>$(find hoverboard_driver)/config/gaz_ros2_ctl_use_sim.yaml</parameters>
+        </plugin>
+    </gazebo>
   </xacro:macro>
 </robot>

File: description/urdf/diffbot.urdf.xacro (robot description, xacro)
@@ -3,9 +3,16 @@
 <robot xmlns:xacro="http://www.ros.org/wiki/xacro" name="diffdrive_robot">
   <xacro:arg name="prefix" default="" />
+  <xacro:arg name="use_ros2_control" default="true"/>
+  <xacro:arg name="sim_mode" default="false"/>
   <xacro:include filename="$(find hoverboard_driver)/urdf/diffbot_description.urdf.xacro" />
   <!-- Import Rviz colors -->
   <xacro:include filename="$(find hoverboard_driver)/urdf/diffbot.materials.xacro" />
   <!-- Import diffbot ros2_control description -->
-  <xacro:include filename="$(find hoverboard_driver)/ros2_control/hoverboard_driver.ros2_control.xacro" />
+  <xacro:if value="$(arg use_ros2_control)">
+    <xacro:include filename="$(find hoverboard_driver)/ros2_control/hoverboard_driver.ros2_control.xacro" />
+  </xacro:if>
+  <xacro:unless value="$(arg use_ros2_control)">
+        <xacro:include filename="gazebo_control.xacro" />
+  </xacro:unless>
   <xacro:diffbot prefix="$(arg prefix)" />
   <xacro:hoverboard_driver_ros2_control

File: description/urdf/diffbot_description.urdf.xacro (robot description, xacro)
@@ -44,5 +44,5 @@
       <parent link="${prefix}base_link"/>
       <child link="${prefix}left_wheel"/>
-      <origin xyz="0 -${base_width/2} ${z_offset}" rpy="0 0 0"/>
+      <origin xyz="0 -0.15 ${z_offset}" rpy="0 0 0"/>
       <axis xyz="0 1 0"/>
       <dynamics damping="0.2"/>
@@ -78,5 +78,5 @@
       <parent link="${prefix}base_link"/>
       <child link="${prefix}right_wheel"/>
-      <origin xyz="0 ${base_width/2} ${z_offset}" rpy="0 0 0"/>
+      <origin xyz="0 0.15 ${z_offset}" rpy="0 0 0"/>
       <axis xyz="0 1 0"/>
       <dynamics damping="0.2"/>

File: description/urdf/lidar.xacro (robot description, xacro)
@@ -4,5 +4,5 @@
   <parent link="${prefix}base_link"/>
   <child link="lidar_link"/>
-  <origin xyz="0.30 0 0.20" rpy="0 0 0"/>
+  <origin xyz="0.30 0 0.20" rpy="0 0 ${PI}"/>
 </joint>
   <link name="lidar_link">

Commit message: coisas

File: description/ros2_control/hoverboard_driver.ros2_control.xacro (robot description, xacro)
@@ -7,5 +7,5 @@
           <plugin>hoverboard_driver/hoverboard_driver</plugin>
           <param name="wheel_radius">0.0825</param>
-          <param name="max_velocity">1.5</param>  <!-- m/s -->
+          <param name="max_velocity">2.0</param>  <!-- m/s -->
           <param name="device">/dev/serial/by-id/usb-Prolific_Technology_Inc._USB-Serial_Controller-if00-port0</param>
         </hardware>

File: description/urdf/lidar.xacro (robot description, xacro)
@@ -4,5 +4,5 @@
   <parent link="${prefix}base_link"/>
   <child link="lidar_link"/>
-  <origin xyz="${base_width/2} 0 -0.023" rpy="0 0 ${PI}"/>
+  <origin xyz="${(base_width/2) + 0.12} 0 -0.023" rpy="0 0 ${PI}"/>
 </joint>
   <link name="lidar_link">
